File: Modul tester.kicad_pcb (KiCad board)
At the start: 2 copper layers, 100 x 100 mm, 11 parts, among them J1 Conn_01x09_Pin, J2 Conn_01x09_Pin, J3 Conn_01x14_Pin, J4 Conn_01x14_Pin, J5 Conn_01x02_Socket, J6 Conn_01x02_Socket, J7 Conn_01x02_Socket

Commit message: 2
Parts:
- added D1: D_Small, Diode_SMD:D_MiniMELF, F.Cu at (124.0, 130.8)
- added D2: LED, LED_SMD:LED_0805_2012Metric, F.Cu at (124.0, 139.9)
- added D3: D_Small, Diode_SMD:D_MiniMELF, F.Cu at (124.0, 106.0)
- added D4: D_Small, Diode_SMD:D_MiniMELF, F.Cu at (124.0, 81.0)
- added D5: D_Small, Diode_SMD:D_MiniMELF, F.Cu at (124.0, 55.8)
- added D6: LED, LED_SMD:LED_0805_2012Metric, F.Cu at (124.0, 114.9)
- added D7: LED, LED_SMD:LED_0805_2012Metric, F.Cu at (124.0, 90.0)
- added D8: LED, LED_SMD:LED_0805_2012Metric, F.Cu at (124.0, 64.9)
- added J10: Conn_01x02_Pin, Connector_PinHeader_2.54mm:PinHeader_1x02_P2.54mm_Vertical, F.Cu at (90.5, 76.0)
- added J11: Conn_01x03_Pin, Connector_PinHeader_2.54mm:PinHeader_1x03_P2.54mm_Vertical, F.Cu at (93.5, 86.0)
- added J8: Conn_02x04_Odd_Even, Connector_PinHeader_2.54mm:PinHeader_2x04_P2.54mm_Vertical, F.Cu at (101.0, 139.5)
- added J9: Conn_01x09_Pin, Connector_Phoenix_MC_HighVoltage:PhoenixContact_MCV_1,5_9-G-5.08_1x09_P5.08mm_Vertical, F.Cu at (82.0, 140.6)
- added R1: R_Small, Resistor_SMD:R_0805_2012Metric, F.Cu at (98.1, 78.0)
- added R2: R_Small, Resistor_SMD:R_0805_2012Metric, F.Cu at (124.0, 135.9)
- added R3: R_Small, Resistor_SMD:R_0805_2012Metric, F.Cu at (124.0, 111.1)
- added R4: R_Small, Resistor_SMD:R_0805_2012Metric, F.Cu at (124.0, 86.1)
- added R5: R_Small, Resistor_SMD:R_0805_2012Metric, F.Cu at (124.0, 61.1)
- moved J5 9.86 mm to (89.2, 56.4)
- moved J6 9.86 mm to (101.7, 56.4)
- moved J7 9.86 mm to (114.7, 56.4)
- moved RV1 2.00 mm to (131.0, 58.0)
- moved RV2 2.00 mm to (131.0, 83.0)
- moved RV3 2.00 mm to (131.0, 108.0)
- moved RV4 2.00 mm to (131.0, 133.0)
Connections:
- J3 pad 13: Y_13 -> Y_1
- J3 pad 6: Y_6 -> Y_1
- J4 pad 13: Y_13 -> Y_1
- J4 pad 6: Y_6 -> Y_1
- J5 pad 1: Y_13 -> Y_1
- J7 pad 2: Y_6 -> Y_1
- RV1 pad 2: unconnected-(RV1-Pad2) -> Y_5
- RV1 pad 3: unconnected-(RV1-Pad3) -> Y_1
- RV2 pad 2: unconnected-(RV2-Pad2) -> Y_4
- RV2 pad 3: unconnected-(RV2-Pad3) -> Y_1
- RV3 pad 2: unconnected-(RV3-Pad2) -> Net-(J11-Pin_1)
- RV3 pad 3: unconnected-(RV3-Pad3) -> Y_1
- RV4 pad 2: unconnected-(RV4-Pad2) -> Y_2
- RV4 pad 3: unconnected-(RV4-Pad3) -> Y_1
Routing:
- net Y_14: track 5.08 -> 181.9 mm
- net Y_5: track 5.08 -> 102.4 mm, vias 0 -> 1
- net Y_2: track 5.08 -> 94.0 mm
- net X_9: track 5.10 -> 82.5 mm
- net X_6: track 5.10 -> 76.6 mm, vias 0 -> 1
- net Y_4: track 5.08 -> 75.4 mm
- net X_4: track 5.10 -> 70.4 mm, vias 0 -> 1
- net Y_7: track 5.08 -> 69.4 mm
- net X_8: track 5.10 -> 68.9 mm
- net X_2: track 5.10 -> 68.7 mm, vias 0 -> 1
- net Net-(J11-Pin_1): track 0.00 -> 47.6 mm
- net X_5: track 5.10 -> 52.4 mm
- net Y_10: track 5.08 -> 50.7 mm
- net Y_9: track 5.08 -> 50.5 mm
- net X_3: track 5.10 -> 42.1 mm
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- added copper zone on B.Cu, net Y_1
- added copper zone on F.Cu, net Y_1
Other:
- board text added: "+"
- board text added: "-"
- board text added: "12 V"
- board text added: "A+"
- board text added: "A/E bus"
- board text added: "B-"
- board text added: "DHW / TPA"
- board text added: "EXT"
- board text added: "EXT / TPM Jumper"
- board text added: "FLOW / TPE"
- board text added: "GND Jumper"
- board text added: "LON"
- board text added: "OUT / TPT"
- board text added: "R1 Jumper"
- board text added: "TPM"
- board text added: "ULM C1 ULM+ PLM+ Tester"
- board text added: "X1 - X2"
- board text added: "X2"
- board text added: "X3 - X4"
- board text added: "X4"
- board text added: "X5 - X6"
- board text added: "X6"
- board text added: "X8 - X9"
- board text added: "X9"
- board text added: "Y2"
- board text added: "Y3"
- board text added: "Y4"
- board text added: "Y5"
