File: Modul tester.kicad_sch (KiCad schematic)
At the start: 11 parts, among them J1 Conn_01x09_Pin, J2 Conn_01x09_Pin, J3 Conn_01x14_Pin, J4 Conn_01x14_Pin, J5 Conn_01x02_Socket, J6 Conn_01x02_Socket, J7 Conn_01x02_Socket

Commit message: 2
Parts:
- added D1, D3, D4, D5: D_Small, Diode_SMD:D_MiniMELF, symbol Device:D_Small
- added D2, D6, D7, D8: LED, LED_SMD:LED_0805_2012Metric, symbol Device:LED
- added J10: Conn_01x02_Pin, Connector_PinHeader_2.54mm:PinHeader_1x02_P2.54mm_Vertical, symbol Connector:Conn_01x02_Pin
- added J11: Conn_01x03_Pin, Connector_PinHeader_2.54mm:PinHeader_1x03_P2.54mm_Vertical, symbol Connector:Conn_01x03_Pin
- added J8: Conn_02x04_Odd_Even, Connector_PinHeader_2.54mm:PinHeader_2x04_P2.54mm_Vertical, symbol Connector_Generic:Conn_02x04_Odd_Even
- added J9: Conn_01x09_Pin, Connector_Phoenix_MC_HighVoltage:PhoenixContact_MCV_1,5_9-G-5.08_1x09_P5.08mm_Vertical, symbol Connector:Conn_01x09_Pin
- added R1, R2, R3, R4, R5: R_Small, Resistor_SMD:R_0805_2012Metric, symbol Device:R_Small
Connections:
- net Y_1 is gone; now on net GND: J3.1 (Pin_1), J4.1 (Pin_1)
- net Y_13 is gone; now on net GND: J3.13 (Pin_13), J4.13 (Pin_13), J5.1 (Pin_1)
- net Y_6 is gone; now on net GND: J3.6 (Pin_6), J4.6 (Pin_6), J7.2 (Pin_2)
- net X_1: now also J8.7 (Pin_7), J9.1 (Pin_1)
- net X_2: now also D2.1 (K), J9.2 (Pin_2)
- net X_3: now also J8.5 (Pin_5), J9.3 (Pin_3)
- net X_4: now also D6.1 (K), J9.4 (Pin_4)
- net X_5: now also J8.3 (Pin_3), J9.5 (Pin_5)
- net X_6: now also D7.1 (K), J9.6 (Pin_6)
- net X_8: now also J8.1 (Pin_1), J9.8 (Pin_8)
- net X_9: now also D8.1 (K), J9.9 (Pin_9)
- net Y_2: now also RV4.2
- net Y_3: now also J11.2 (Pin_2)
- net Y_4: now also RV2.2
- net Y_5: now also RV1.2, J10.1 (Pin_1), J10.2 (Pin_2), R1.1, R1.2
- net at RV3.2: now also J11.1 (Pin_1)
- net GND: now reaches RV3.3
- net GND: now also RV1.3, RV2.3, RV4.3, J11.3 (Pin_3), J8.2 (Pin_2), J8.4 (Pin_4), J8.6 (Pin_6), J8.8 (Pin_8)
- net Y_14 renamed +12V
- net +12V: now also D1.1 (K), D1.2 (A), D3.1 (K), D3.2 (A), D4.1 (K), D4.2 (A), D5.1 (K), D5.2 (A), R2.1, R3.1, R4.1, R5.1
- new net: D6.2 (A), R3.2
- new net: D7.2 (A), R4.2
- new net: D2.2 (A), R2.2
- new net: D8.2 (A), R5.2
- no-connect marks 6 -> 11
